File: arm_modified_pcb/arm_pcb.kicad_pcb (KiCad board)
At the start: 2 copper layers, 91.4 x 69 mm, 21 parts, among them U1 NODEMCU32S

Commit message: Arm/Ld Modified
Parts:
- added CanBus_PowerSwitch: InputSwitch, Connector_PinHeader_2.54mm:PinHeader_1x03_P2.54mm_Vertical, F.Cu at (224.5, 107.6)
- added Canbus: CanBUS, Connector_PinSocket_2.54mm:PinSocket_1x04_P2.54mm_Horizontal, F.Cu at (200.0, 105.1)
- moved I2Cbreakout1 4.99 mm to (157.8, 102.9)
- moved Servo1 2.68 mm to (177.0, 118.5)
- moved Servo2 2.68 mm to (192.2, 118.5)
- moved Servo3 2.68 mm to (207.4, 118.5)
- moved Servo4 2.68 mm to (222.7, 118.5)
Connections:
- U1 pad GPIO10: unconnected-(U1-PadGPIO10) -> Net-(J1-Pin_1)
- U1 pad GPIO9: unconnected-(U1-PadGPIO9) -> Net-(J1-Pin_2)
Routing:
- net Net-(J1-Pin_1): track 0.00 -> 62.3 mm, vias 0 -> 1
- net Net-(J1-Pin_2): track 0.00 -> 60.9 mm
- net Net-(J1-Pin_4): track 0.00 -> 26.9 mm
- net VCCQ: track 277.5 -> 289.5 mm
- net GND: track 31.4 -> 27.4 mm, vias 8 -> 17
- net Net-(Servo2-Pin_2): track 37.4 -> 40.1 mm
- net Net-(Servo1-Pin_2): track 27.2 -> 29.2 mm
- net VCC: track 156.6 -> 157.9 mm
- net GPIO5: track 99.3 -> 100.1 mm
