File: arm_modified_pcb/arm_pcb.kicad_pcb (KiCad board)
At the start: 2 copper layers, 91.4 x 69 mm, 23 parts, among them U1 NODEMCU32S

Commit message: Few Small Changes
Routing:
- net GND: track 27.4 -> 19.7 mm, vias 17 -> 42
- net VCCQ: track 289.5 -> 287.4 mm
- net SPI_MOSI: track 71.7 -> 70.9 mm
- net tx: track 59.9 -> 59.2 mm
- net rx: track 55.9 -> 55.2 mm
- net SPI_RST: track 21.0 -> 20.3 mm
- net a_in_1: track 44.7 -> 44.2 mm

Commit message: Add files via upload
Connections:
- Servo1 pad 1: GND -> Net-(Servo1-Pin_1)
- Servo1 pad 2: Net-(Servo1-Pin_2) -> VCC
- Servo1 pad 3: VCC -> GND
- Servo2 pad 1: GND -> Net-(Servo2-Pin_1)
- Servo2 pad 2: Net-(Servo2-Pin_2) -> VCC
- Servo2 pad 3: VCC -> GND
- Servo3 pad 1: GND -> servo3
- Servo3 pad 2: servo3 -> VCC
- Servo3 pad 3: VCC -> GND
- Servo4 pad 1: GND -> servo4
- Servo4 pad 2: servo4 -> VCC
- Servo4 pad 3: VCC -> GND
- U1 pad GPIO16: Net-(Servo2-Pin_2) -> Net-(Servo2-Pin_1)
- U1 pad GPIO17: Net-(Servo1-Pin_2) -> Net-(Servo1-Pin_1)
Routing:
- net Net-(Servo2-Pin_1): track 0.00 -> 41.2 mm
- net Net-(Servo2-Pin_2): track 40.1 -> 0.00 mm
- net Net-(Servo1-Pin_1): track 0.00 -> 29.2 mm
- net Net-(Servo1-Pin_2): track 29.2 -> 0.00 mm
- net VCC: track 157.9 -> 154.6 mm
- net servo4: track 90.4 -> 92.9 mm
- net servo3: track 70.2 -> 71.3 mm
