File: arm_modified_pcb/arm_pcb.kicad_sch (KiCad schematic)
At the start: 17 parts, among them U1 NODEMCU32S

Commit message: Add files via upload
Connections:
- net GND: now also Servo1.3 (Pin_3), Servo2.3 (Pin_3), Servo3.3 (Pin_3), Servo4.3 (Pin_3); no longer Servo1.1 (Pin_1), Servo2.1 (Pin_1), Servo3.1 (Pin_1), Servo4.1 (Pin_1)
- net VCC: now also Servo1.2 (Pin_2), Servo2.2 (Pin_2), Servo3.2 (Pin_2), Servo4.2 (Pin_2); no longer Servo1.3 (Pin_3), Servo2.3 (Pin_3), Servo3.3 (Pin_3), Servo4.3 (Pin_3)
- net servo3: now also Servo3.1 (Pin_1); no longer Servo3.2 (Pin_2)
- net servo4: now also Servo4.1 (Pin_1); no longer Servo4.2 (Pin_2)
- net at U1.GPIO16: now also Servo2.1 (Pin_1); no longer Servo2.2 (Pin_2)
- net at U1.GPIO17: now also Servo1.1 (Pin_1); no longer Servo1.2 (Pin_2)
