File: MainPCB/MainPCB.kicad_pcb (KiCad board)
At the start: 2 copper layers, 50 parts, among them J1 esp1_jst1, J10 Raspi_pinout4, J11 Raspi_pinout5, J12 esp2_jst2, J13 esp2_jst3, J14 Conn_01x02_Pin, J15 esp2_jst1, J16 esp2_jst4, J17 esp3_pinout1, J18 esp3_pinout4, J19 Conn_01x02_Pin, J2 esp1_jst2, J20 esp3_pinout3, J21 esp3_pinout2, J22 esp4_pinout3, J23 esp4_pinout2, J24 Conn_01x02_Pin, J25 esp4_pinout1, J26 esp4_pinout4, J27 esp5_pinout3, J28 esp5_pinout2, J29 Conn_01x02_Pin, J3 esp1_jst3, J30 esp5_pinout1, J31 esp5_pinout4, J32 I2C_in1, J33 I2C_Out1, J34 I2C_in2, J35 I2C_Out2, J4 esp1_jst4, J5 Raspi_pinout1, J6 Raspi_pinout2, J7 Raspi_pinout3, J8 Conn_01x02_Pin, J9 Raspi_pinout6

Commit message: Add files via upload
Parts:
- moved J9 28.5 mm to (235.0, 64.5), turned to 180 degrees
- moved Esp3 23.1 mm to (211.1, 132.4)
- moved EspCan3 9.13 mm to (198.5, 102.3)
- moved EspCan5 5.20 mm to (227.5, 145.2)
- moved J11 5.16 mm to (242.4, 44.4)
- moved Esp5 4.39 mm to (226.7, 158.7)
- moved J10 3.92 mm to (242.3, 72.6)
- moved J6 3.51 mm to (235.1, 72.5)
Changed lines of the file:
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@@
 	(footprint "Connector_PinHeader_2.54mm:PinHeader_1x02_P2.54mm_Vertical"
 		(layer "F.Cu")
-		(at 228.35 150.345)
+		(at 227.5 145.21)
 		(descr "Through hole straight pin header, 1x02, 2.54mm pitch, single row")
 		(tags "Through hole pin header THT 1x02 2.54mm single row")
@@
 	(footprint "Connector_PinHeader_2.54mm:PinHeader_1x08_P2.54mm_Vertical"
 		(layer "F.Cu")
-		(at 238.36 72.97)
+		(at 242.26 72.6)
 		(descr "Through hole straight pin header, 1x08, 2.54mm pitch, single row")
 		(tags "Through hole pin header THT 1x08 2.54mm single row")
@@
 	(footprint "Connector_PinHeader_2.54mm:PinHeader_1x08_P2.54mm_Vertical"
 		(layer "F.Cu")
-		(at 231.68 71.65)
+		(at 235.08 72.52)
 		(descr "Through hole straight pin header, 1x08, 2.54mm pitch, single row")
 		(tags "Through hole pin header THT 1x08 2.54mm single row")
@@
 	(footprint "Connector_PinHeader_2.54mm:PinHeader_1x02_P2.54mm_Vertical"
 		(layer "F.Cu")
-		(at 205.82 96.83)
+		(at 198.48 102.255)
 		(descr "Through hole straight pin header, 1x02, 2.54mm pitch, single row")
 		(tags "Through hole pin header THT 1x02 2.54mm single row")
@@
 	(footprint "Connector_PinHeader_2.54mm:PinHeader_1x09_P2.54mm_Vertical"
 		(layer "F.Cu")
-		(at 237.62 42.5)
+		(at 242.41 44.41)
 		(descr "Through hole straight pin header, 1x09, 2.54mm pitch, single row")
 		(tags "Through hole pin header THT 1x09 2.54mm single row")
@@
 	(footprint "Connector_PinSocket_2.54mm:PinSocket_2x10_P2.54mm_Vertical"
 		(layer "F.Cu")
-		(at 192.2 119.01 180)
+		(at 211.06 132.43 180)
 		(descr "Through hole straight socket strip, 2x10, 2.54mm pitch, double cols (from Kicad 4.0.7), script generated")
 		(tags "Through hole socket strip THT 2x10 2.54mm double row")
@@
 	(footprint "Connector_PinSocket_2.54mm:PinSocket_2x10_P2.54mm_Vertical"
 		(layer "F.Cu")
-		(at 229.83 161.7 -90)
+		(at 226.66 158.67 -90)
 		(descr "Through hole straight socket strip, 2x10, 2.54mm pitch, double cols (from Kicad 4.0.7), script generated")
 		(tags "Through hole socket strip THT 2x10 2.54mm double row")
@@
 	(footprint "Connector_PinHeader_2.54mm:PinHeader_1x09_P2.54mm_Vertical"
 		(layer "F.Cu")
-		(at 239.03 36.27 -90)
+		(at 235.01 64.52 180)
 		(descr "Through hole straight pin header, 1x09, 2.54mm pitch, single row")
 		(tags "Through hole pin header THT 1x09 2.54mm single row")
 		(property "Reference" "J9"
-			(at 0 -2.33 90)
+			(at 0 -2.33 0)
 			(layer "F.SilkS")
 			(effects
@@
 		)
 		(property "Value" "Raspi_pinout6"
-			(at 0 22.65 90)
+			(at 0 22.65 0)
 			(layer "F.Fab")
 			(effects
@@
 		)
 		(property "Footprint" "Connector_PinHeader_2.54mm:PinHeader_1x09_P2.54mm_Vertical"
-			(at 0 0 -90)
+			(at 0 0 180)
 			(unlocked yes)
 			(layer "F.Fab")
@@
 		)
 		(property "Datasheet" ""
-			(at 0 0 -90)
+			(at 0 0 180)
 			(unlocked yes)
 			(layer "F.Fab")
@@
 		)
 		(property "Description" "Generic connector, single row, 01x09, script generated"
-			(at 0 0 -90)
+			(at 0 0 180)
 			(unlocked yes)
 			(layer "F.Fab")
@@
 		(attr through_hole)
 		(fp_line
-			(start -1.33 21.65)
+			(start 1.33 1.27)
 			(end 1.33 21.65)
 			(stroke
@@
 		)
 		(fp_line
-			(start -1.33 1.27)
-			(end -1.33 21.65)
+			(start -1.33 21.65)
+			(end 1.33 21.65)
 			(stroke
 				(width 0.12)
@@
 		)
 		(fp_line
-			(start 1.33 1.27)
-			(end 1.33 21.65)
+			(start -1.33 1.27)
+			(end -1.33 21.65)
 			(stroke
 				(width 0.12)
@@
 		)
 		(fp_line
-			(start -1.8 22.1)
-			(end 1.8 22.1)
+			(start 1.8 22.1)
+			(end 1.8 -1.8)
 			(stroke
 				(width 0.05)
@@
 		)
 		(fp_line
-			(start 1.8 22.1)
-			(end 1.8 -1.8)
+			(start 1.8 -1.8)
+			(end -1.8 -1.8)
 			(stroke
 				(width 0.05)
@@
 		)
 		(fp_line
-			(start -1.8 -1.8)
-			(end -1.8 22.1)
+			(start -1.8 22.1)
+			(end 1.8 22.1)
 			(stroke
 				(width 0.05)
@@
 		)
 		(fp_line
-			(start 1.8 -1.8)
-			(end -1.8 -1.8)
+			(start -1.8 -1.8)
+			(end -1.8 22.1)
 			(stroke
 				(width 0.05)
@@
 		)
 		(fp_line
-			(start -1.27 21.59)
-			(end -1.27 -0.635)
+			(start 1.27 21.59)
+			(end -1.27 21.59)
 			(stroke
 				(width 0.1)
@@
 		)
 		(fp_line
-			(start 1.27 21.59)
-			(end -1.27 21.59)
+			(start 1.27 -1.27)
+			(end 1.27 21.59)
 			(stroke
 				(width 0.1)
@@
 		)
 		(fp_line
-			(start -1.27 -0.635)
-			(end -0.635 -1.27)
+			(start -0.635 -1.27)
+			(end 1.27 -1.27)
 			(stroke
 				(width 0.1)
@@
 		)
 		(fp_line
-			(start -0.635 -1.27)
-			(end 1.27 -1.27)
+			(start -1.27 21.59)
+			(end -1.27 -0.635)
 			(stroke
 				(width 0.1)
@@
 		)
 		(fp_line
-			(start 1.27 -1.27)
-			(end 1.27 21.59)
+			(start -1.27 -0.635)
+			(end -0.635 -1.27)
 			(stroke
 				(width 0.1)
@@
 		)
 		(fp_text user "${REFERENCE}"
-			(at 0 10.16 0)
+			(at 0 10.16 90)
 			(layer "F.Fab")
 			(effects
@@
 		)
 		(pad "1" thru_hole rect
-			(at 0 0 270)
+			(at 0 0 180)
 			(size 1.7 1.7)
 			(drill 1)
@@
 		)
 		(pad "2" thru_hole oval
-			(at 0 2.54 270)
+			(at 0 2.54 180)
 			(size 1.7 1.7)
 			(drill 1)
@@
 		)
 		(pad "3" thru_hole oval
-			(at 0 5.08 270)
+			(at 0 5.08 180)
 			(size 1.7 1.7)
 			(drill 1)
@@
 		)
 		(pad "4" thru_hole oval
-			(at 0 7.62 270)
+			(at 0 7.62 180)
 			(size 1.7 1.7)
 			(drill 1)
@@
 		)
 		(pad "5" thru_hole oval
-			(at 0 10.16 270)
+			(at 0 10.16 180)
 			(size 1.7 1.7)
 			(drill 1)
@@
 		)
 		(pad "6" thru_hole oval
-			(at 0 12.7 270)
+			(at 0 12.7 180)
 			(size 1.7 1.7)
 			(drill 1)
@@
 		)
 		(pad "7" thru_hole oval
-			(at 0 15.24 270)
+			(at 0 15.24 180)
 			(size 1.7 1.7)
 			(drill 1)
@@
 		)
 		(pad "8" thru_hole oval
-			(at 0 17.78 270)
+			(at 0 17.78 180)
 			(size 1.7 1.7)
 			(drill 1)
@@
 		)
 		(pad "9" thru_hole oval
-			(at 0 20.32 270)
+			(at 0 20.32 180)
 			(size 1.7 1.7)
 			(drill 1)

Commit message: Add files via upload
Parts:
- removed J14, J19, J24, J29: Conn_01x02_Pin, Connector_PinHeader_2.54mm:PinHeader_1x02_P2.54mm_Vertical
- added 12V_3: XT60-M, Connector_AMASS:AMASS_XT60-M_1x02_P7.20mm_Vertical, F.Cu at (70.4, 87.7)
- added 12V_4: XT60-M, Connector_AMASS:AMASS_XT60-M_1x02_P7.20mm_Vertical, F.Cu at (70.4, 97.9)
- added 5V_3: XT60-M, Connector_AMASS:AMASS_XT60-M_1x02_P7.20mm_Vertical, F.Cu at (69.9, 130.0)
- added 5V_4: XT60-M, Connector_AMASS:AMASS_XT60-M_1x02_P7.20mm_Vertical, F.Cu at (70.4, 118.4)
- J8: value Conn_01x02_Pin -> Conn_01x08_Pin; footprint Connector_PinHeader_2.54mm:PinHeader_1x02_P2.54mm_Vertical -> Connector_PinHeader_2.54mm:PinHeader_1x08_P2.54mm_Vertical
- moved EspCan5 173.8 mm to (93.4, 34.7)
- moved J30 152.4 mm to (156.9, 16.9), turned to 90 degrees
- moved Esp3 146.3 mm to (103.0, 33.8), turned to 90 degrees
- moved Esp5 144.0 mm to (153.9, 34.4), turned to 90 degrees
- moved J28 142.5 mm to (172.3, 21.9), turned to -90 degrees
- moved J17 140.6 mm to (75.1, 33.8), turned to 180 degrees
- moved J31 138.3 mm to (152.1, 17.4), turned to -90 degrees
- moved J21 137.0 mm to (101.2, 18.0)
- moved J27 131.8 mm to (152.0, 22.7), turned to -90 degrees
- moved J32 120.9 mm to (89.1, 59.0)
- moved J34 120.9 mm to (89.1, 66.2)
- moved J33 119.1 mm to (73.3, 63.4)
- moved J26 100.6 mm to (247.4, 89.3), turned to 180 degrees
- moved J25 98.4 mm to (247.9, 143.5)
- moved J22 97.2 mm to (247.4, 119.7)
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Connections:
- Esp1 pad 14: Net-(Esp1-Pin_14) -> esp1_pin3
- Esp1 pad 16: Net-(Esp1-Pin_16) -> esp1_pin2
- Esp1 pad 18: Net-(Esp1-Pin_18) -> esp1_pin1
- J1 pad 1: unconnected-(J1-Pin_1-Pad1) -> GND
- J10 pad 6: unconnected-(J10-Pin_6-Pad6) -> GND
- J10 pad 7: unconnected-(J10-Pin_7-Pad7) -> 5V_4
- J10 pad 8: unconnected-(J10-Pin_8-Pad8) -> 12V_3
- J11 pad 8: unconnected-(J11-Pin_8-Pad8) -> 5V_4
- J11 pad 9: unconnected-(J11-Pin_9-Pad9) -> 12V_3
- J12 pad 1: unconnected-(J12-Pin_1-Pad1) -> GND
- J13 pad 1: unconnected-(J13-Pin_1-Pad1) -> GND
- J15 pad 1: unconnected-(J15-Pin_1-Pad1) -> GND
- J16 pad 1: unconnected-(J16-Pin_1-Pad1) -> GND
- J17 pad 1: unconnected-(J17-Pin_1-Pad1) -> 12V_1
- J17 pad 2: unconnected-(J17-Pin_2-Pad2) -> GND
- J17 pad 7: unconnected-(J17-Pin_7-Pad7) -> 5V_1
- J18 pad 1: unconnected-(J18-Pin_1-Pad1) -> 12V_1
- J18 pad 2: unconnected-(J18-Pin_2-Pad2) -> GND
- J18 pad 7: unconnected-(J18-Pin_7-Pad7) -> 5V_1
- J2 pad 1: unconnected-(J2-Pin_1-Pad1) -> GND
- J20 pad 1: unconnected-(J20-Pin_1-Pad1) -> 12V_1
- J20 pad 2: unconnected-(J20-Pin_2-Pad2) -> GND
- J20 pad 7: unconnected-(J20-Pin_7-Pad7) -> 5V_1
- J21 pad 1: unconnected-(J21-Pin_1-Pad1) -> 12V_1
- J21 pad 2: unconnected-(J21-Pin_2-Pad2) -> GND
- J21 pad 7: unconnected-(J21-Pin_7-Pad7) -> 5V_1
- J22 pad 1: unconnected-(J22-Pin_1-Pad1) -> 12V_2
- J22 pad 2: unconnected-(J22-Pin_2-Pad2) -> GND
- J22 pad 7: unconnected-(J22-Pin_7-Pad7) -> 5V_2
- J23 pad 1: unconnected-(J23-Pin_1-Pad1) -> 12V_2
- J23 pad 2: unconnected-(J23-Pin_2-Pad2) -> GND
- J23 pad 7: unconnected-(J23-Pin_7-Pad7) -> 5V_2
- J25 pad 1: unconnected-(J25-Pin_1-Pad1) -> 12V_2
- J25 pad 2: unconnected-(J25-Pin_2-Pad2) -> GND
- J25 pad 7: unconnected-(J25-Pin_7-Pad7) -> 5V_2
- J26 pad 1: unconnected-(J26-Pin_1-Pad1) -> 12V_2
- J26 pad 2: unconnected-(J26-Pin_2-Pad2) -> GND
- J26 pad 7: unconnected-(J26-Pin_7-Pad7) -> 5V_2
- J27 pad 1: unconnected-(J27-Pin_1-Pad1) -> 12V_2
- J27 pad 2: unconnected-(J27-Pin_2-Pad2) -> GND
- J27 pad 7: unconnected-(J27-Pin_7-Pad7) -> 5V_3
- J28 pad 1: unconnected-(J28-Pin_1-Pad1) -> 12V_2
- J28 pad 2: unconnected-(J28-Pin_2-Pad2) -> GND
- J28 pad 7: unconnected-(J28-Pin_7-Pad7) -> 5V_3
- J3 pad 1: unconnected-(J3-Pin_1-Pad1) -> GND
- J30 pad 1: unconnected-(J30-Pin_1-Pad1) -> 12V_2
- J30 pad 2: unconnected-(J30-Pin_2-Pad2) -> GND
- J30 pad 7: unconnected-(J30-Pin_7-Pad7) -> 5V_3
- J31 pad 1: unconnected-(J31-Pin_1-Pad1) -> 12V_2
- J31 pad 2: unconnected-(J31-Pin_2-Pad2) -> GND
- J31 pad 7: unconnected-(J31-Pin_7-Pad7) -> 5V_3
- J33 pad 1: unconnected-(J33-Pin_1-Pad1) -> 12V_2
- J33 pad 5: unconnected-(J33-Pin_5-Pad5) -> 5V_3
- J35 pad 1: unconnected-(J35-Pin_1-Pad1) -> 12V_2
- J35 pad 5: unconnected-(J35-Pin_5-Pad5) -> 5V_3
- J4 pad 1: unconnected-(J4-Pin_1-Pad1) -> GND
- J4 pad 3: Net-(Esp1-Pin_14) -> esp1_pin3
- J4 pad 4: Net-(Esp1-Pin_16) -> esp1_pin2
- J4 pad 5: Net-(Esp1-Pin_18) -> esp1_pin1
- J5 pad 7: unconnected-(J5-Pin_7-Pad7) -> 5V_4
- J5 pad 8: unconnected-(J5-Pin_8-Pad8) -> 12V_3
- J6 pad 7: unconnected-(J6-Pin_7-Pad7) -> 5V_4
- J6 pad 8: unconnected-(J6-Pin_8-Pad8) -> 12V_3
- J7 pad 7: unconnected-(J7-Pin_7-Pad7) -> 5V_4
- J7 pad 8: unconnected-(J7-Pin_8-Pad8) -> 12V_3
- J8 pad 1: rx -> 12V_4
- J8 pad 2: tx -> GND
- J9 pad 8: unconnected-(J9-Pin_8-Pad8) -> 5V_4
- J9 pad 9: unconnected-(J9-Pin_9-Pad9) -> 12V_3

Commit message: Add files via upload
Parts:
- removed 12V_4: XT60-M, Connector_AMASS:AMASS_XT60-M_1x02_P7.20mm_Vertical
- removed J10: Raspi_pinout4, Connector_PinHeader_2.54mm:PinHeader_1x08_P2.54mm_Vertical
- removed J18: esp3_pinout4, Connector_PinHeader_2.54mm:PinHeader_1x07_P2.54mm_Vertical
- removed J8: Conn_01x08_Pin, Connector_PinHeader_2.54mm:PinHeader_1x08_P2.54mm_Vertical
- added Jee1: esp3_pinout4, Connector_PinHeader_2.54mm:PinHeader_1x07_P2.54mm_Vertical, F.Cu at (270.5, 36.8)
- Esp3: value Fan_and_temperature -> Drive
- Esp5: value Extra1 -> Fans
- moved EspCan5 275.4 mm to (327.5, 179.8), turned to 180 degrees
- moved J30 257.5 mm to (359.3, 176.0), turned to 180 degrees
- moved J28 247.9 mm to (359.3, 184.7), turned to 0 degrees
- moved J31 246.6 mm to (358.6, 152.2), turned to 180 degrees
- moved Esp5 231.5 mm to (339.8, 172.3), turned to 180 degrees
- moved J27 226.0 mm to (358.6, 114.1), turned to 0 degrees
- moved J17 216.6 mm to (291.7, 36.7), turned to -90 degrees
- moved J21 200.9 mm to (299.1, 52.1), turned to 180 degrees
- moved J16 182.6 mm to (296.4, 184.7)
- moved Esp3 181.8 mm to (281.6, 67.8), turned to -90 degrees
- moved J34 178.1 mm to (262.2, 108.0), turned to 180 degrees
- moved J32 169.2 mm to (251.0, 108.0), turned to 90 degrees
- moved J33 159.3 mm to (231.7, 47.0), turned to 180 degrees
- moved J2 155.3 mm to (263.2, 84.7)
- moved J13 142.1 mm to (309.6, 140.0), turned to 90 degrees
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Connections:
- 12V_1 pad 1: (no net) -> 12V_1
- 12V_1 pad 2: (no net) -> GND
- 12V_2 pad 1: (no net) -> 12V_2
- 12V_2 pad 2: (no net) -> GND
- 12V_3 pad 1: (no net) -> 12V_3
- 12V_3 pad 2: (no net) -> GND
- 5V_1 pad 1: (no net) -> 5V_1
- 5V_1 pad 2: (no net) -> GND
- 5V_2 pad 1: (no net) -> 5V_2
- 5V_2 pad 2: (no net) -> GND
- 5V_3 pad 1: (no net) -> 5V_3
- 5V_3 pad 2: (no net) -> GND
- 5V_4 pad 1: (no net) -> 5V_4
- 5V_4 pad 2: (no net) -> GND
- Esp1 pad 14: esp1_pin3 -> Net-(Esp1-Pin_14)
- Esp1 pad 16: esp1_pin2 -> Net-(Esp1-Pin_16)
- Esp1 pad 18: esp1_pin1 -> Net-(Esp1-Pin_18)
- Esp1 pad 19: unconnected-(Esp1-Pin_19-Pad19) -> GND
- Esp1 pad 20: unconnected-(Esp1-Pin_20-Pad20) -> 5V_1
- Esp2 pad 19: unconnected-(Esp2-Pin_19-Pad19) -> GND
- Esp2 pad 20: unconnected-(Esp2-Pin_20-Pad20) -> 5V_1
- Esp3 pad 19: unconnected-(Esp3-Pin_19-Pad19) -> GND
- Esp3 pad 20: unconnected-(Esp3-Pin_20-Pad20) -> 5V_1
- Esp4 pad 19: unconnected-(Esp4-Pin_19-Pad19) -> GND
- Esp4 pad 20: unconnected-(Esp4-Pin_20-Pad20) -> 5V_1
- Esp5 pad 19: unconnected-(Esp5-Pin_19-Pad19) -> GND
- Esp5 pad 20: unconnected-(Esp5-Pin_20-Pad20) -> 5V_1
- J1 pad 1: GND -> Net-(Esp1-Pin_10)
- J1 pad 2: Net-(Esp1-Pin_4) -> Net-(Esp1-Pin_8)
- J1 pad 4: Net-(Esp1-Pin_8) -> Net-(Esp1-Pin_4)
- J1 pad 5: Net-(Esp1-Pin_10) -> GND
- J11 pad 1: GPIO_16 -> GPIO_13
- J11 pad 2: GPIO_17 -> GPIO_6
- J11 pad 3: GPIO_18 -> GPIO_5
- J11 pad 4: GPIO_19 -> GPIO_0
- J11 pad 5: GPIO_20 -> GPIO_11
- J11 pad 6: GPIO_21 -> GPIO_9
- J12 pad 1: GND -> Net-(Esp2-Pin_2)
- J12 pad 2: Net-(Esp2-Pin_5) -> Net-(Esp2-Pin_1)
- J12 pad 4: Net-(Esp2-Pin_1) -> Net-(Esp2-Pin_5)
- J12 pad 5: Net-(Esp2-Pin_2) -> GND
- J13 pad 1: GND -> Net-(Esp2-Pin_13)
- J13 pad 2: Net-(Esp2-Pin_7) -> Net-(Esp2-Pin_11)
- J13 pad 4: Net-(Esp2-Pin_11) -> Net-(Esp2-Pin_7)
- J13 pad 5: Net-(Esp2-Pin_13) -> GND
- J15 pad 1: GND -> Net-(Esp2-Pin_10)
- J15 pad 2: Net-(Esp2-Pin_4) -> Net-(Esp2-Pin_8)
- J15 pad 4: Net-(Esp2-Pin_8) -> Net-(Esp2-Pin_4)
- J15 pad 5: Net-(Esp2-Pin_10) -> GND
- J16 pad 1: GND -> Net-(Esp2-Pin_18)
- J16 pad 2: Net-(Esp2-Pin_12) -> Net-(Esp2-Pin_16)
- J16 pad 4: Net-(Esp2-Pin_16) -> Net-(Esp2-Pin_12)
- J16 pad 5: Net-(Esp2-Pin_18) -> GND
- J2 pad 1: GND -> Net-(Esp1-Pin_2)
- J2 pad 2: Net-(Esp1-Pin_5) -> Net-(Esp1-Pin_1)
- J2 pad 4: Net-(Esp1-Pin_1) -> Net-(Esp1-Pin_5)
- J2 pad 5: Net-(Esp1-Pin_2) -> GND
- J3 pad 1: GND -> Net-(Esp1-Pin_13)
- J3 pad 2: Net-(Esp1-Pin_7) -> Net-(Esp1-Pin_11)
- J3 pad 4: Net-(Esp1-Pin_11) -> Net-(Esp1-Pin_7)
- J3 pad 5: Net-(Esp1-Pin_13) -> GND
- J4 pad 1: GND -> Net-(Esp1-Pin_12)
- J4 pad 2: Net-(Esp1-Pin_12) -> Net-(Esp1-Pin_14)
- J4 pad 3: esp1_pin3 -> Net-(Esp1-Pin_16)
- J4 pad 4: esp1_pin2 -> Net-(Esp1-Pin_18)
- J4 pad 5: esp1_pin1 -> GND
- J5 pad 1: GPIO_24 -> GPIO_14
- J5 pad 2: GPIO_0 -> GPIO_15
- J5 pad 3: GPIO_1 -> GPIO_18
- J5 pad 4: GPIO_2 -> GPIO_23
- J5 pad 5: GPIO_3 -> GPIO_24
- J6 pad 1: GPIO_7 -> GPIO_25
- J6 pad 3: GPIO_9 -> GPIO_7
- J6 pad 4: GPIO_10 -> GPIO_1
- J6 pad 5: GPIO_11 -> GPIO_12
- J7 pad 1: GPIO_26 -> GPIO_16
- J7 pad 2: GPIO_12 -> GPIO_20
- J7 pad 3: GPIO_13 -> GPIO_21
- J7 pad 4: GPIO_14 -> GPIO_26
- J7 pad 5: GPIO_15 -> GPIO_19
- J9 pad 1: GPIO_22 -> GPIO_10
- J9 pad 2: GPIO_23 -> GPIO_22
- J9 pad 3: GPIO_24 -> GPIO_27
- J9 pad 4: GPIO_25 -> GPIO_17
- J9 pad 5: GPIO_26 -> GPIO_4
- J9 pad 6: GPIO_27 -> GPIO_3
- Raspi1 pad 1: unconnected-(Raspi1-Pin_1-Pad1) -> 3.3v
- Raspi1 pad 17: unconnected-(Raspi1-Pin_17-Pad17) -> 3.3v
- Raspi1 pad 2: VCC -> 5V_4
- Raspi1 pad 3: GPIO_2 -> unconnected-(Raspi1-Pin_3-Pad3)
- Raspi1 pad 4: VCC -> 5V_4
Routing:
- net 5V_3: track 0.00 -> 424.8 mm
- net Net-(EspCan1-Pin_1): track 0.00 -> 300.7 mm
- net Net-(EspCan1-Pin_2): track 0.00 -> 297.2 mm
- net 5V_4: track 0.00 -> 243.6 mm
- net tx: track 0.00 -> 195.0 mm, vias 0 -> 2
- net rx: track 0.00 -> 192.1 mm, vias 0 -> 3
- net 5V_2: track 0.00 -> 130.8 mm
- net Net-(J34-Pin_2): track 0.00 -> 75.4 mm
- net Net-(J32-Pin_4): track 0.00 -> 75.1 mm
- net Net-(J34-Pin_4): track 0.00 -> 74.6 mm
- net Net-(Esp1-Pin_5): track 0.00 -> 71.9 mm
- net Net-(J32-Pin_2): track 0.00 -> 71.5 mm
- net Net-(Esp1-Pin_1): track 0.00 -> 69.0 mm
- net Net-(Esp1-Pin_3): track 0.00 -> 66.8 mm
- net Net-(Esp4-Pin_7): track 0.00 -> 63.9 mm
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Other:
- board outline added: 230 x 175 mm
