File: MainPCB/MainPCB.kicad_sch (KiCad schematic)
At the start: 45 parts, among them J1 esp1_jst1, J10 Raspi_pinout4, J11 Raspi_pinout5, J12 esp2_jst2, J13 esp2_jst3, J15 esp2_jst1, J16 esp2_jst4, J17 esp3_pinout1, J18 esp3_pinout4, J2 esp1_jst2, J20 esp3_pinout3, J21 esp3_pinout2, J22 esp4_pinout3, J23 esp4_pinout2, J25 esp4_pinout1, J26 esp4_pinout4, J27 esp5_pinout3, J28 esp5_pinout2, J3 esp1_jst3, J30 esp5_pinout1, J31 esp5_pinout4, J32 I2C_in1, J33 I2C_Out1, J34 I2C_in2, J35 I2C_Out2, J4 esp1_jst4, J5 Raspi_pinout1, J6 Raspi_pinout2, J7 Raspi_pinout3, J9 Raspi_pinout6

Commit message: Add files via upload
Parts:
- added 12V_3, 5V_3, 5V_4: XT60-M, Connector_AMASS:AMASS_XT60-M_1x02_P7.20mm_Vertical, symbol XT60-M:XT60-M
Connections:
- net 12V_1: now also J17.1 (Pin_1), J18.1 (Pin_1), J20.1 (Pin_1), J21.1 (Pin_1)
- net 12V_2: now also J22.1 (Pin_1), J23.1 (Pin_1), J25.1 (Pin_1), J26.1 (Pin_1), J27.1 (Pin_1), J28.1 (Pin_1), J30.1 (Pin_1), J31.1 (Pin_1), J33.1 (Pin_1), J35.1 (Pin_1)
- net 5V_1: now also J17.7 (Pin_7), J18.7 (Pin_7), J20.7 (Pin_7), J21.7 (Pin_7)
- net 5V_2: now also J22.7 (Pin_7), J23.7 (Pin_7), J25.7 (Pin_7), J26.7 (Pin_7)
- net GND: now also J1.1 (Pin_1), J10.6 (Pin_6), J12.1 (Pin_1), J13.1 (Pin_1), J15.1 (Pin_1), J16.1 (Pin_1), J17.2 (Pin_2), J18.2 (Pin_2), J2.1 (Pin_1), J20.2 (Pin_2), J21.2 (Pin_2), J22.2 (Pin_2), J23.2 (Pin_2), J25.2 (Pin_2), J26.2 (Pin_2), J27.2 (Pin_2), J28.2 (Pin_2), J3.1 (Pin_1), J30.2 (Pin_2), J31.2 (Pin_2), J4.1 (Pin_1), 12V_3.N (NEG), 5V_3.N (NEG), 5V_4.N (NEG)
- net 5V_4: now reaches J5.7 (Pin_7)
- net 5V_4: now also J10.7 (Pin_7), J11.8 (Pin_8), J6.7 (Pin_7), J7.7 (Pin_7), J9.8 (Pin_8), 5V_4.P (POS)
- net 12V_3: now reaches J5.8 (Pin_8)
- net 12V_3: now also J10.8 (Pin_8), J11.9 (Pin_9), J6.8 (Pin_8), J7.8 (Pin_8), J9.9 (Pin_9), 12V_3.P (POS)
- net 5V_3: now reaches J35.5 (Pin_5)
- net 5V_3: now also J27.7 (Pin_7), J28.7 (Pin_7), J30.7 (Pin_7), J31.7 (Pin_7), J33.5 (Pin_5), 5V_3.P (POS)

Commit message: Add files via upload
Parts:
- added 12V_4: XT60-M, Connector_AMASS:AMASS_XT60-M_1x02_P7.20mm_Vertical, symbol XT60-M:XT60-M
- added J8: Conn_01x08_Pin, Connector_PinHeader_2.54mm:PinHeader_1x08_P2.54mm_Vertical, symbol Connector:Conn_01x08_Pin
Connections:
- net GND: now also 12V_4.N (NEG), J8.2 (Pin_2)
- net esp1_pin3: now reaches Esp1.14 (Pin_14), J4.3 (Pin_3)
- net esp1_pin3: now also J8.5 (Pin_5)
- net esp1_pin2: now reaches Esp1.16 (Pin_16), J4.4 (Pin_4)
- net esp1_pin2: now also J8.4 (Pin_4)
- net esp1_pin1: now reaches Esp1.18 (Pin_18), J4.5 (Pin_5)
- net esp1_pin1: now also J8.3 (Pin_3)
- new net 12V_4: 12V_4.P (POS), J8.1 (Pin_1)

Commit message: Add files via upload
Parts:
- removed 12V_4: XT60-M, Connector_AMASS:AMASS_XT60-M_1x02_P7.20mm_Vertical, symbol XT60-M:XT60-M
- removed J10: Raspi_pinout4, Connector_PinHeader_2.54mm:PinHeader_1x08_P2.54mm_Vertical, symbol Connector:Conn_01x08_Socket
- removed J8: Conn_01x08_Pin, Connector_PinHeader_2.54mm:PinHeader_1x08_P2.54mm_Vertical, symbol Connector:Conn_01x08_Pin
- Esp3: value Fan_and_temperature -> Drive
- Esp5: value Extra1 -> Fans
- EspCan1, EspCan2, EspCan3, EspCan4, EspCan5: symbol Connector:Conn_01x02_Pin -> Connector:Conn_01x02_Male
- J1, J12, J13, J15, J16, J2, J3, J33, J35, J4: symbol Connector:Conn_01x05_Pin -> Connector:Conn_01x05_Male
- J11, J9: symbol Connector:Conn_01x09_Socket -> Connector:Conn_01x09_Female
- J17, J20, J21, J22, J23, J25, J26, J27, J28, J30, J31: symbol Connector:Conn_01x07_Pin -> Connector:Conn_01x07_Male
- J5, J6, J7: symbol Connector:Conn_01x08_Socket -> Connector:Conn_01x08_Female
- Jee1: renamed from J18; symbol Connector:Conn_01x07_Pin -> Connector:Conn_01x07_Male
Connections:
- net VCC is gone; now on net 5V_4: Raspi1.2 (Pin_2), Raspi1.4 (Pin_4)
- net 12V_1: now also 12V_1.1 (P); no longer 12V_1.P (POS)
- net 12V_2: now also 12V_2.1 (P); no longer 12V_2.P (POS)
- net 12V_3: now also 12V_3.1 (P); no longer 12V_3.P (POS)
- net 5V_1: now also 5V_1.1 (P), Esp1.20 (Pin_20), Esp2.20 (Pin_20), Esp3.20 (Pin_20), Esp4.20 (Pin_20), Esp5.20 (Pin_20); no longer 5V_1.P (POS)
- net 5V_2: now also 5V_2.1 (P); no longer 5V_2.P (POS)
- net 5V_3: now also 5V_3.1 (P); no longer 5V_3.P (POS)
- net 5V_4: now also 5V_4.1 (P); no longer 5V_4.P (POS)
- net GND: now also 12V_1.2 (N), 12V_2.2 (N), 12V_3.2 (N), 5V_1.2 (N), 5V_2.2 (N), 5V_3.2 (N), 5V_4.2 (N), Esp1.19 (Pin_19), Esp2.19 (Pin_19), Esp3.19 (Pin_19), Esp4.19 (Pin_19), Esp5.19 (Pin_19), J1.5 (Pin_5), J12.5 (Pin_5), J13.5 (Pin_5), J15.5 (Pin_5), J16.5 (Pin_5), J2.5 (Pin_5), J3.5 (Pin_5), J4.5 (Pin_5); no longer 12V_1.N (NEG), 12V_2.N (NEG), 12V_3.N (NEG), 5V_1.N (NEG), 5V_2.N (NEG), 5V_3.N (NEG), 5V_4.N (NEG), J1.1 (Pin_1), J12.1 (Pin_1), J13.1 (Pin_1), J15.1 (Pin_1), J16.1 (Pin_1), J2.1 (Pin_1), J3.1 (Pin_1), J4.1 (Pin_1)
- net GPIO_0: now also J11.4 (Pin_4); no longer J5.2 (Pin_2)
- net GPIO_1: now also J6.4 (Pin_4); no longer J5.3 (Pin_3)
- net GPIO_10: now also J9.1 (Pin_1); no longer J6.4 (Pin_4)
- net GPIO_11: now also J11.5 (Pin_5); no longer J6.5 (Pin_5)
- net GPIO_12: now also J6.5 (Pin_5); no longer J7.2 (Pin_2)
- net GPIO_13: now also J11.1 (Pin_1); no longer J7.3 (Pin_3)
- net GPIO_14: now also J5.1 (Pin_1); no longer J7.4 (Pin_4)
- net GPIO_15: now also J5.2 (Pin_2); no longer J7.5 (Pin_5)
- net GPIO_16: now also J7.1 (Pin_1); no longer J11.1 (Pin_1)
- net GPIO_17: now also J9.4 (Pin_4); no longer J11.2 (Pin_2)
- net GPIO_18: now also J5.3 (Pin_3); no longer J11.3 (Pin_3)
- net GPIO_19: now also J7.5 (Pin_5); no longer J11.4 (Pin_4)
- net GPIO_20: now also J7.2 (Pin_2); no longer J11.5 (Pin_5)
- net GPIO_21: now also J7.3 (Pin_3); no longer J11.6 (Pin_6)
- net GPIO_22: now also J9.2 (Pin_2); no longer J9.1 (Pin_1)
- net GPIO_23: now also J5.4 (Pin_4); no longer J9.2 (Pin_2)
- net GPIO_24: now also J5.5 (Pin_5); no longer J5.1 (Pin_1), J9.3 (Pin_3)
- net GPIO_25: now also J6.1 (Pin_1); no longer J9.4 (Pin_4)
- net GPIO_26: now also J7.4 (Pin_4); no longer J7.1 (Pin_1), J9.5 (Pin_5)
- net GPIO_27: now also J9.3 (Pin_3); no longer J9.6 (Pin_6)
- net GPIO_3: now also J9.6 (Pin_6); no longer J5.5 (Pin_5)
- net GPIO_4: now also J9.5 (Pin_5)
- net GPIO_5: now also J11.3 (Pin_3)
- net GPIO_6: now also J11.2 (Pin_2)
- net GPIO_7: now also J6.3 (Pin_3); no longer J6.1 (Pin_1)
- net GPIO_9: now also J11.6 (Pin_6); no longer J6.3 (Pin_3)
- net at J13.2 (Pin_2): now also Esp2.11 (Pin_11); no longer Esp2.7 (Pin_7)
- net at J13.4 (Pin_4): now also Esp2.7 (Pin_7); no longer Esp2.11 (Pin_11)
- net at Esp2.13 (Pin_13): now also J13.1 (Pin_1); no longer J13.5 (Pin_5)
- net at J16.2 (Pin_2): now also Esp2.16 (Pin_16); no longer Esp2.12 (Pin_12)
- net at J16.4 (Pin_4): now also Esp2.12 (Pin_12); no longer Esp2.16 (Pin_16)
- net at Esp2.18 (Pin_18): now also J16.1 (Pin_1); no longer J16.5 (Pin_5)
- net at J1.2 (Pin_2): now also Esp1.8 (Pin_8); no longer Esp1.4 (Pin_4)
- net at J1.4 (Pin_4): now also Esp1.4 (Pin_4); no longer Esp1.8 (Pin_8)
- net at Esp1.10 (Pin_10): now also J1.1 (Pin_1); no longer J1.5 (Pin_5)
- net at J15.2 (Pin_2): now also Esp2.8 (Pin_8); no longer Esp2.4 (Pin_4)
- net at J15.4 (Pin_4): now also Esp2.4 (Pin_4); no longer Esp2.8 (Pin_8)
- net at Esp2.10 (Pin_10): now also J15.1 (Pin_1); no longer J15.5 (Pin_5)
- net at J3.2 (Pin_2): now also Esp1.11 (Pin_11); no longer Esp1.7 (Pin_7)
- net at J3.4 (Pin_4): now also Esp1.7 (Pin_7); no longer Esp1.11 (Pin_11)
- net at Esp1.13 (Pin_13): now also J3.1 (Pin_1); no longer J3.5 (Pin_5)
- net at J12.2 (Pin_2): now also Esp2.1 (Pin_1); no longer Esp2.5 (Pin_5)
- net at J12.4 (Pin_4): now also Esp2.5 (Pin_5); no longer Esp2.1 (Pin_1)
- net at Esp2.2 (Pin_2): now also J12.1 (Pin_1); no longer J12.5 (Pin_5)
- net 3.3v: now reaches Raspi1.1 (Pin_1)
- net 3.3v: now also Raspi1.17 (Pin_17)
- net at Esp1.1 (Pin_1): now also J2.2 (Pin_2); no longer J2.4 (Pin_4)
- net at Esp1.12 (Pin_12): now also J4.1 (Pin_1); no longer J4.2 (Pin_2)
- net at Esp1.2 (Pin_2): now also J2.1 (Pin_1); no longer J2.5 (Pin_5)
- net at Esp1.5 (Pin_5): now also J2.4 (Pin_4); no longer J2.2 (Pin_2)
- net GPIO_2: no longer names the net of Raspi1.3 (Pin_3)
- net GPIO_2: no longer J5.4 (Pin_4)
- net esp1_pin1: no longer names the net of Esp1.18 (Pin_18)
- net esp1_pin1: now also J4.4 (Pin_4); no longer J4.5 (Pin_5)
- net esp1_pin2: no longer names the net of Esp1.16 (Pin_16)
- net esp1_pin2: now also J4.3 (Pin_3); no longer J4.4 (Pin_4)
- net esp1_pin3: no longer names the net of Esp1.14 (Pin_14)
- net esp1_pin3: now also J4.2 (Pin_2); no longer J4.3 (Pin_3)
- no-connect marks 0 -> 1
Other:
- moved on the sheet: J1, J15, J16, J3, J32, J33, J34, J35, J4
